File: adc/ADC Wing Board.sch (EAGLE design)
At the start: 28 parts, among them U1 ADS7947SRTET

Commit message: Add switch for choosing between built in GND or REFGND
Parts:
- removed GND, NC1, NC2, NC3: (no value), pinhead:PINHD-1X1
- added REFG: (no value), pinhead:PINHD-1X1
- added S1: (no value), switch:255SB
Connections:
- new net N$2: S1.P, U1.REFGND
- new net N$4: REFG.1, S1.S
- net GND: now also JP1.1, S1.O; no longer GND.1, U1.REFGND
Other:
- moved on the sheet: JP1
Changed lines of the file:
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@@
 <part name="U1" library="ADS7947" deviceset="ADS7947SRTET" device=""/>
 <part name="REF" library="pinhead" library_urn="urn:adsk.eagle:library:325" deviceset="PINHD-1X1" device="" package3d_urn="urn:adsk.eagle:package:22485/2"/>
-<part name="GND" library="pinhead" library_urn="urn:adsk.eagle:library:325" deviceset="PINHD-1X1" device="" package3d_urn="urn:adsk.eagle:package:22485/2"/>
 <part name="AVDD" library="pinhead" library_urn="urn:adsk.eagle:library:325" deviceset="PINHD-1X1" device="" package3d_urn="urn:adsk.eagle:package:22485/2"/>
 <part name="IN0" library="pinhead" library_urn="urn:adsk.eagle:library:325" deviceset="PINHD-1X1" device="" package3d_urn="urn:adsk.eagle:package:22485/2"/>
@@
 <part name="R2" library="rcl" library_urn="urn:adsk.eagle:library:334" deviceset="R-US_" device="R0805" package3d_urn="urn:adsk.eagle:package:23553/2" value="5 Ohm"/>
 <part name="R5" library="rcl" library_urn="urn:adsk.eagle:library:334" deviceset="R-US_" device="R0805" package3d_urn="urn:adsk.eagle:package:23553/2" value="47 Ohm"/>
-<part name="NC1" library="pinhead" library_urn="urn:adsk.eagle:library:325" deviceset="PINHD-1X1" device="" package3d_urn="urn:adsk.eagle:package:22485/2"/>
-<part name="NC2" library="pinhead" library_urn="urn:adsk.eagle:library:325" deviceset="PINHD-1X1" device="" package3d_urn="urn:adsk.eagle:package:22485/2"/>
-<part name="NC3" library="pinhead" library_urn="urn:adsk.eagle:library:325" deviceset="PINHD-1X1" device="" package3d_urn="urn:adsk.eagle:package:22485/2"/>
 <part name="FRAME1" library="frames" library_urn="urn:adsk.eagle:library:229" deviceset="A4L-LOC" device=""/>
 <part name="GND1" library="supply1" library_urn="urn:adsk.eagle:library:371" deviceset="GND" device=""/>
@@
 <part name="GND3" library="supply1" library_urn="urn:adsk.eagle:library:371" deviceset="GND" device=""/>
 <part name="GND4" library="supply1" library_urn="urn:adsk.eagle:library:371" deviceset="GND" device=""/>
-<part name="GND6" library="supply1" library_urn="urn:adsk.eagle:library:371" deviceset="GND" device=""/>
 <part name="GND5" library="supply1" library_urn="urn:adsk.eagle:library:371" deviceset="GND" device=""/>
 <part name="GND7" library="supply1" library_urn="urn:adsk.eagle:library:371" deviceset="GND" device=""/>
@@
 <part name="JP1" library="pinhead" library_urn="urn:adsk.eagle:library:325" deviceset="PINHD-1X8" device="" package3d_urn="urn:adsk.eagle:package:22409/2"/>
 <part name="JP2" library="pinhead" library_urn="urn:adsk.eagle:library:325" deviceset="PINHD-1X8" device="" package3d_urn="urn:adsk.eagle:package:22409/2"/>
+<part name="S1" library="switch" library_urn="urn:adsk.eagle:library:380" deviceset="255SB" device="" package3d_urn="urn:adsk.eagle:package:27679/1"/>
+<part name="GND9" library="supply1" library_urn="urn:adsk.eagle:library:371" deviceset="GND" device=""/>
+<part name="REFG" library="pinhead" library_urn="urn:adsk.eagle:library:325" deviceset="PINHD-1X1" device="" package3d_urn="urn:adsk.eagle:package:22485/2"/>
 </parts>
 <sheets>
@@
 <attribute name="VALUE" x="-36.83" y="91.44" size="1.778" layer="96" rot="R180"/>
 </instance>
-<instance part="GND" gate="G$1" x="-43.18" y="104.14" smashed="yes" rot="R180">
-<attribute name="NAME" x="-36.83" y="100.965" size="1.778" layer="95" rot="R180"/>
-<attribute name="VALUE" x="-36.83" y="109.22" size="1.778" layer="96" rot="R180"/>
-</instance>
 <instance part="AVDD" gate="G$1" x="-43.18" y="73.66" smashed="yes" rot="R180">
 <attribute name="NAME" x="-36.83" y="70.485" size="1.778" layer="95" rot="R180"/>
@@
 <attribute name="NAME" x="138.43" y="54.3814" size="1.778" layer="95" rot="R180"/>
 <attribute name="VALUE" x="138.43" y="59.182" size="1.778" layer="96" rot="R180"/>
-</instance>
-<instance part="NC1" gate="G$1" x="63.5" y="93.98" smashed="yes" rot="R180">
-<attribute name="NAME" x="69.85" y="90.805" size="1.778" layer="95" rot="R180"/>
-<attribute name="VALUE" x="69.85" y="99.06" size="1.778" layer="96" rot="R180"/>
-</instance>
-<instance part="NC2" gate="G$1" x="63.5" y="104.14" smashed="yes" rot="R180">
-<attribute name="NAME" x="69.85" y="100.965" size="1.778" layer="95" rot="R180"/>
-<attribute name="VALUE" x="69.85" y="109.22" size="1.778" layer="96" rot="R180"/>
-</instance>
-<instance part="NC3" gate="G$1" x="63.5" y="114.3" smashed="yes" rot="R180">
-<attribute name="NAME" x="69.85" y="111.125" size="1.778" layer="95" rot="R180"/>
-<attribute name="VALUE" x="69.85" y="119.38" size="1.778" layer="96" rot="R180"/>
 </instance>
 <instance part="FRAME1" gate="G$1" x="-73.66" y="-33.02" smashed="yes">
@@
 <attribute name="VALUE" x="30.48" y="86.36" size="1.778" layer="96" rot="R180"/>
 </instance>
-<instance part="GND2" gate="1" x="22.86" y="104.14" smashed="yes" rot="R90">
-<attribute name="VALUE" x="25.4" y="101.6" size="1.778" layer="96" rot="R90"/>
+<instance part="GND2" gate="1" x="15.24" y="104.14" smashed="yes" rot="R90">
+<attribute name="VALUE" x="17.78" y="101.6" size="1.778" layer="96" rot="R90"/>
 </instance>
 <instance part="GND3" gate="1" x="-15.24" y="25.4" smashed="yes" rot="R270">
@@
 <instance part="GND4" gate="1" x="-15.24" y="-2.54" smashed="yes" rot="R270">
 <attribute name="VALUE" x="-17.78" y="0" size="1.778" layer="96" rot="R270"/>
-</instance>
-<instance part="GND6" gate="1" x="20.32" y="83.82" smashed="yes" rot="R180">
-<attribute name="VALUE" x="22.86" y="86.36" size="1.778" layer="96" rot="R180"/>
 </instance>
 <instance part="GND5" gate="1" x="109.22" y="22.86" smashed="yes">
@@
 <attribute name="VALUE" x="3.556" y="92.329" size="1.778" layer="96"/>
 </instance>
-<instance part="JP1" gate="A" x="-38.1" y="27.94" smashed="yes" rot="R180">
-<attribute name="NAME" x="-31.75" y="14.605" size="1.778" layer="95" rot="R180"/>
-<attribute name="VALUE" x="-31.75" y="40.64" size="1.778" layer="96" rot="R180"/>
+<instance part="JP1" gate="A" x="-50.8" y="114.3" smashed="yes" rot="R180">
+<attribute name="NAME" x="-44.45" y="100.965" size="1.778" layer="95" rot="R180"/>
+<attribute name="VALUE" x="-44.45" y="127" size="1.778" layer="96" rot="R180"/>
 </instance>
 <instance part="JP2" gate="A" x="165.1" y="55.88" smashed="yes">
 <attribute name="NAME" x="158.75" y="69.215" size="1.778" layer="95"/>
 <attribute name="VALUE" x="158.75" y="43.18" size="1.778" layer="96"/>
+</instance>
+<instance part="S1" gate="1" x="17.78" y="96.52" smashed="yes">
+<attribute name="NAME" x="11.43" y="94.615" size="1.778" layer="95" rot="R90"/>
+<attribute name="VALUE" x="13.97" y="99.695" size="1.778" layer="96" rot="R90"/>
+</instance>
+<instance part="GND9" gate="1" x="12.7" y="116.84" smashed="yes" rot="R180">
+<attribute name="VALUE" x="15.24" y="119.38" size="1.778" layer="96" rot="R180"/>
+</instance>
+<instance part="REFG" gate="G$1" x="27.94" y="119.38" smashed="yes" rot="R90">
+<attribute name="NAME" x="24.765" y="113.03" size="1.778" layer="95" rot="R90"/>
+<attribute name="VALUE" x="33.02" y="113.03" size="1.778" layer="96" rot="R90"/>
 </instance>
 </instances>
@@
 </segment>
 <segment>
-<pinref part="GND" gate="G$1" pin="1"/>
-<wire x1="-40.64" y1="104.14" x2="-30.48" y2="104.14" width="0.1524" layer="91"/>
+<wire x1="-48.26" y1="104.14" x2="-30.48" y2="104.14" width="0.1524" layer="91"/>
 <wire x1="-30.48" y1="99.06" x2="-30.48" y2="104.14" width="0.1524" layer="91"/>
 <junction x="-30.48" y="104.14"/>
@@
 <pinref part="GND2" gate="1" pin="GND"/>
 <wire x1="-5.08" y1="104.14" x2="2.54" y2="104.14" width="0.1524" layer="91"/>
-<wire x1="2.54" y1="104.14" x2="20.32" y2="104.14" width="0.1524" layer="91"/>
+<wire x1="2.54" y1="104.14" x2="12.7" y2="104.14" width="0.1524" layer="91"/>
 <wire x1="-5.08" y1="99.06" x2="-5.08" y2="104.14" width="0.1524" layer="91"/>
 <junction x="-5.08" y="104.14"/>
@@
 <pinref part="C5" gate="G$1" pin="1"/>
 <pinref part="C6" gate="G$1" pin="1"/>
-</segment>
-<segment>
-<pinref part="U1" gate="A" pin="REFGND"/>
-<wire x1="33.02" y1="58.42" x2="20.32" y2="58.42" width="0.1524" layer="91"/>
-<pinref part="GND6" gate="1" pin="GND"/>
-<wire x1="20.32" y1="58.42" x2="20.32" y2="81.28" width="0.1524" layer="91"/>
+<pinref part="JP1" gate="A" pin="1"/>
 </segment>
 <segment>
@@
 <wire x1="99.06" y1="60.96" x2="99.06" y2="71.12" width="0.1524" layer="91"/>
 <pinref part="GND8" gate="1" pin="GND"/>
+</segment>
+<segment>
+<pinref part="S1" gate="1" pin="O"/>
+<wire x1="17.78" y1="101.6" x2="17.78" y2="109.22" width="0.1524" layer="91"/>
+<wire x1="17.78" y1="109.22" x2="12.7" y2="109.22" width="0.1524" layer="91"/>
+<pinref part="GND9" gate="1" pin="GND"/>
+<wire x1="12.7" y1="109.22" x2="12.7" y2="114.3" width="0.1524" layer="91"/>
 </segment>
 </net>
@@
 </segment>
 </net>
+<net name="N$2" class="0">
+<segment>
+<pinref part="U1" gate="A" pin="REFGND"/>
+<wire x1="33.02" y1="58.42" x2="20.32" y2="58.42" width="0.1524" layer="91"/>
+<pinref part="S1" gate="1" pin="P"/>
+<wire x1="20.32" y1="58.42" x2="20.32" y2="91.44" width="0.1524" layer="91"/>
+</segment>
+</net>
+<net name="N$4" class="0">
+<segment>
+<pinref part="S1" gate="1" pin="S"/>
+<wire x1="22.86" y1="101.6" x2="22.86" y2="109.22" width="0.1524" layer="91"/>
+<wire x1="22.86" y1="109.22" x2="27.94" y2="109.22" width="0.1524" layer="91"/>
+<pinref part="REFG" gate="G$1" pin="1"/>
+<wire x1="27.94" y1="109.22" x2="27.94" y2="116.84" width="0.1524" layer="91"/>
+</segment>
+</net>
